File: pcb_hs/chilineko-pcb.sch (KiCad schematic (older format))
At the start: 20 parts, among them J1 JST SH 4-pin, J2 AVR-ISP-6, J3 DATA Breakout, J4 VBUS Breakout, SW1 Reset, U1 SRV05-4, U2 ATmega32U4-AU, Y1 16MHz

Commit message: Update lib references
Parts:
- J2: symbol chilineko-pcb-rescue:AVR-ISP-6-Connector-bakeneko-65-pcb-rescue-hs_bakeneko-65-pcb-rescue-hs_bakeneko-65-pcb-rescue -> Arduino:AVR-ISP-6-Connector
- U2: symbol chilineko-pcb-rescue:ATmega32U4-AU-MCU_Microchip_ATmega-bakeneko-65-pcb-rescue-hs_bakeneko-65-pcb-rescue-hs_bakeneko-65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 -> Arduino:ATmega32U4-AU-MCU_Microchip_ATmega
Changed lines of the file:
@@
 D+
 $Comp
-L chilineko-pcb-rescue:ATmega32U4-AU-MCU_Microchip_ATmega-bakeneko-65-pcb-rescue-hs_bakeneko-65-pcb-rescue-hs_bakeneko-65-pcb-rescue U2
+L Arduino:ATmega32U4-AU-MCU_Microchip_ATmega U2
 U 1 1 5F26004F
 P 2300 5050
@@
 	5350 5150 5650 5150
 $Comp
-L chilineko-pcb-rescue:AVR-ISP-6-Connector-bakeneko-65-pcb-rescue-hs_bakeneko-65-pcb-rescue-hs_bakeneko-65-pcb-rescue J2
+L Arduino:AVR-ISP-6-Connector J2
 U 1 1 5F4C9CCE
 P 2050 1700
